File: charging and protection/CP/CP.kicad_pcb (KiCad board)
At the start: 2 copper layers, 53.2 x 23.4 mm, 6 parts, among them J1 Screw_Terminal_01x02, J2 Screw_Terminal_01x02, J3 Screw_Terminal_01x02, J4 Screw_Terminal_01x02, J5 Screw_Terminal_01x02, U1 TP4056_MICRO-USB_CHARGER_-_1A

Commit message: refresh
Routing:
- removed copper zone on B.Cu, net (none)
Changed lines of the file:
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@@
 		(pad "1" thru_hole roundrect
 			(at 0 0 270)
-			(size 1.7 2)
+			(size 2 2)
 			(drill 1)
 			(layers "*.Cu" "*.Mask")
@@
 		(pad "1" thru_hole roundrect
 			(at 0 0 270)
-			(size 1.7 2)
+			(size 2 2)
 			(drill 1)
 			(layers "*.Cu" "*.Mask")
@@
 		(end 105.82 87.85)
 		(width 2)
-		(locked yes)
 		(layer "F.Cu")
 		(net 1)
@@
 		(end 113.25 87.85)
 		(width 2)
-		(locked yes)
 		(layer "F.Cu")
 		(net 4)
-	)
-	(zone
-		(net 7)
-		(net_name "VCC")
-		(layer "F.Cu")
-		(hatch edge 0.5)
-		(connect_pads yes
-			(clearance 0.5)
-		)
-		(min_thickness 0.25)
-		(filled_areas_thickness no)
-		(fill yes
-			(thermal_gap 0.5)
-			(thermal_bridge_width 0.5)
-		)
-		(polygon
-			(pts
-				(xy 122.92 96.94) (xy 118.78 95.56) (xy 104.78 97.13) (xy 104.83 91.84) (xy 93.62 91.94) (xy 93.05 107.58)
-				(xy 122.9 104.28)
-			)
-		)
 	)
 	(zone
@@
 	)
 	(zone
+		(net 7)
+		(net_name "VCC")
+		(layer "F.Cu")
+		(hatch edge 0.5)
+		(connect_pads yes
+			(clearance 0.8)
+		)
+		(min_thickness 0.25)
+		(filled_areas_thickness no)
+		(fill yes
+			(thermal_gap 0)
+			(thermal_bridge_width 0.5)
+		)
+		(polygon
+			(pts
+				(xy 122.92 96.94) (xy 118.78 95.56) (xy 104.78 97.13) (xy 104.83 91.84) (xy 93.62 91.94) (xy 93.05 107.58)
+				(xy 122.9 104.28)
+			)
+		)
+	)
+	(zone
 		(net 8)
 		(net_name "GND")
@@
 		(hatch edge 0.5)
 		(connect_pads yes
-			(clearance 0.5)
+			(clearance 0.8)
 		)
 		(min_thickness 0.25)
@@
 		)
 	)
-	(zone
-		(net 0)
-		(net_name "")
-		(layer "B.Cu")
-		(hatch edge 0.5)
-		(priority 1)
-		(connect_pads yes
-			(clearance 0.5)
-		)
-		(min_thickness 0.25)
-		(filled_areas_thickness no)
-		(fill yes
-			(thermal_gap 0.5)
-			(thermal_bridge_width 0.5)
-			(island_removal_mode 1)
-			(island_area_min 10)
-		)
-		(polygon
-			(pts
-				(xy 199.74 35.3) (xy 37.21 31.85) (xy 44.26 147.59) (xy 203.05 145.72)
-			)
-		)
-	)
-	(group ""
-		(locked yes)
-		(members "0965be72-946b-4169-b3f0-a3d94e317ff3" "1ca7bf4d-d64d-41e5-a7f6-9af896936edc"
-			"2270ca7b-678a-4c05-860c-6b68eacfa954" "23d3a056-a24d-44fc-8c78-8e26871670f1"
-			"31a96dc3-7760-4735-89c0-8bc70de11708" "3e6e7a37-3b3a-434f-abd5-9f7cdccf7623"
-			"4dc26adc-eb97-4882-ba7d-30e469b8ae49" "58677aa3-1d43-4fff-a737-ebf7518ba9d7"
-			"5ff91e41-2431-4def-86af-dbe6a1db3ad5" "76eb7485-1995-4bb3-9485-0e7b5d58c198"
-			"7ec5ba8f-f72d-4207-a5d3-7aa01499d70b" "a6587e3e-3456-476c-b2f8-a574ed7b304e"
-			"bbf91fc5-c638-4a5a-b399-36d40dc42dc0" "c4572dd4-4983-4d6e-9454-4801fb8a0b44"
-			"c52140e1-7f5e-4228-b58d-2572675569c7" "d5e26fd8-dc2b-4a6c-972b-5d4ccefc236a"
-			"dd4c212e-ecab-4848-8988-24f2e8d08c91" "e8f14b1d-90e7-496d-8033-6301293b7c4b"
-			"f1e5ba17-f8a6-453e-91b8-58623cdbfd7b" "f24150bb-0492-4ba6-9ff9-3c7a1f82c175"
-		)
-	)

Commit message: refresh
Parts:
- J5: footprint Connector_AMASS:AMASS_XT30U-F_1x02_P5.0mm_Vertical -> Connector_AMASS:AMASS_XT30PW-M_1x02_P2.50mm_Horizontal
- moved J5 4.29 mm to (99.1, 89.6)
Routing:
- removed copper zone on F.Cu, net GND
- removed copper zone on F.Cu, net VCC
Other:
- board size 53.2 x 23.4 mm -> 62.6 x 23.4 mm
