File: microcontroller/micro/micro.kicad_pcb (KiCad board)
At the start: 2 copper layers, 60 x 60 mm, 21 parts, among them J1 USB_C_Receptacle_USB2.0_16P, U1 STM32F405RGTx, U2 TPD4E05U06DQA

Commit message: refresh
Parts:
- moved FB1 11.2 mm to (147.8, 79.8)
Routing:
- net Net-(J1-VBUS-PadA4): track 27.7 -> 30.4 mm

Commit message: refresh
Parts:
- added J2: Screw_Terminal_01x03, Connector_JST:JST_EH_B3B-EH-A_1x03_P2.50mm_Vertical, B.Cu at (164.2, 122.0)
- moved C13 2.20 mm to (151.9, 101.0)
Routing:
- net GND: track 90.4 -> 0.77 mm, vias 0 -> 3
- net Net-(J2-Pin_2): track 0.00 -> 0.76 mm, vias 0 -> 5
- added copper zone on In1.Cu, net GND
- added copper zone on In2.Cu, net Net-(J2-Pin_2)
Other:
- copper layers 2 -> 4

Commit message: refresh
Routing:
- net GND: track 0.77 -> 53.5 mm
- net /USB_+: track 18.7 -> 15.7 mm
- net /USB_-: track 18.6 -> 15.7 mm

Commit message: refresh
Parts:
- C11, C13, C4, C5, C7, C9: footprint Capacitor_Tantalum_SMD:CP_EIA-1608-08_AVX-J -> Capacitor_Tantalum_SMD:CP_EIA-6032-28_Kemet-C
- FB1: footprint Ferrite_THT:LairdTech_28C0236-0JW-10 -> Inductor_SMD:L_Walsin_WLFM201609x
- moved C2 38.0 mm to (177.4, 109.7), turned to -90 degrees
- moved C10 37.7 mm to (180.4, 89.9)
- moved C1 35.3 mm to (180.4, 87.5)
- moved C8 31.6 mm to (175.1, 109.7), turned to -90 degrees
- moved C9 31.4 mm to (181.3, 93.7)
- moved C7 28.6 mm to (171.2, 110.7), turned to -90 degrees
- moved C5 26.4 mm to (164.8, 110.7), turned to -90 degrees
- moved C12 23.3 mm to (159.9, 88.5), turned to 90 degrees
- moved C6 20.7 mm to (160.9, 109.7), turned to -90 degrees
- moved FB1 18.6 mm to (157.5, 95.8)
- moved C11 16.8 mm to (163.8, 87.5), turned to 90 degrees
- moved C4 9.72 mm to (149.3, 95.8), turned to 180 degrees
- moved C14 6.69 mm to (150.3, 105.6), turned to 180 degrees
- moved C3 5.34 mm to (150.3, 92.0), turned to 180 degrees
- moved C13 2.68 mm to (149.3, 101.8), turned to 180 degrees
Connections:
- C10 pad 1: Net-(J2-Pin_2) -> Net-(C10-Pad1)
- C11 pad 1: Net-(J2-Pin_2) -> Net-(C11-Pad1)
- C12 pad 1: Net-(J2-Pin_2) -> Net-(C11-Pad1)
- C13 pad 1: Net-(J2-Pin_2) -> Net-(U1-VDDA)
- C14 pad 1: Net-(J2-Pin_2) -> Net-(U1-VDDA)
- C3 pad 1: Net-(J2-Pin_2) -> Net-(C3-Pad1)
- C4 pad 1: Net-(J2-Pin_2) -> Net-(C3-Pad1)
- C5 pad 1: Net-(J2-Pin_2) -> Net-(C5-Pad1)
- C6 pad 1: Net-(J2-Pin_2) -> Net-(C5-Pad1)
- C7 pad 1: Net-(J2-Pin_2) -> Net-(C7-Pad1)
- C8 pad 1: Net-(J2-Pin_2) -> Net-(C7-Pad1)
- C9 pad 1: Net-(J2-Pin_2) -> Net-(C10-Pad1)
- FB1 pad 1: Net-(J2-Pin_2) -> Net-(C3-Pad1)
- J2 pad 2: Net-(J2-Pin_2) -> unconnected-(J2-Pin_2-Pad2)
- U1 pad 13: Net-(J2-Pin_2) -> Net-(U1-VDDA)
- U1 pad 19: Net-(J2-Pin_2) -> Net-(C5-Pad1)
- U1 pad 32: Net-(J2-Pin_2) -> Net-(C7-Pad1)
- U1 pad 48: Net-(J2-Pin_2) -> Net-(C10-Pad1)
- U1 pad 64: Net-(J2-Pin_2) -> Net-(C11-Pad1)
Routing:
- net GND: track 53.5 -> 148.6 mm
- net Net-(U1-VCAP_2): track 0.00 -> 15.6 mm
- net Net-(U1-VDDA): track 0.00 -> 13.9 mm, vias 0 -> 1
- net Net-(U1-VCAP_1): track 0.00 -> 11.1 mm
- net Net-(C10-Pad1): track 0.00 -> 10.5 mm, vias 0 -> 1
- net Net-(C3-Pad1): track 0.00 -> 8.34 mm
- net Net-(C11-Pad1): track 0.00 -> 7.62 mm, vias 0 -> 1
- net Net-(C7-Pad1): track 0.00 -> 6.87 mm, vias 0 -> 1
- net Net-(C5-Pad1): track 0.00 -> 6.87 mm, vias 0 -> 1
- net Net-(U1-VBAT): track 0.00 -> 3.19 mm
- net /USB_-: track 15.7 -> 16.5 mm
- net /USB_+: track 15.7 -> 16.4 mm
- net unconnected-(J2-Pin_2-Pad2): track 0.00 -> 0.76 mm
- net Net-(J2-Pin_2): track 0.76 -> 0.00 mm, vias 5 -> 0
- added copper zone on In2.Cu, net unconnected-(J2-Pin_2-Pad2)
- removed copper zone on In2.Cu, net Net-(J2-Pin_2)

Commit message: refresh
Routing:
- net GND: track 148.6 -> 68.0 mm, vias 3 -> 2
- net Net-(U1-VDDA): track 13.9 -> 17.1 mm
- net Net-(C7-Pad1): track 6.87 -> 8.56 mm
- net Net-(C5-Pad1): track 6.87 -> 8.56 mm
- net Net-(C3-Pad1): track 8.34 -> 9.99 mm, vias 0 -> 1
- net Net-(C10-Pad1): track 10.5 -> 11.6 mm

Commit message: refresh
Parts:
- moved R3 0.33 mm to (181.7, 100.4)
Routing:
- net Net-(U1-VCAP_2): track 15.6 -> 13.7 mm
- net Net-(J1-CC2): track 13.7 -> 15.5 mm

Commit message: refresh
Routing:
- net Net-(C11-Pad1): track 7.62 -> 9.31 mm
