File: microcontroller/micro/micro.kicad_pcb (KiCad board)
At the start: 4 copper layers, 60 x 60 mm, 22 parts, among them J1 USB_C_Receptacle_USB2.0_16P, J2 Screw_Terminal_01x03, U1 STM32F405RGTx, U2 TPD4E05U06DQA

Commit message: refresh
Routing:
- net GND: track 68.0 -> 118.2 mm, vias 2 -> 4
- net Net-(U1-VDDA): track 17.1 -> 15.6 mm

Commit message: refresh
Parts:
- moved U2 0.75 mm to (181.5, 98.2), turned to 180 degrees
Connections:
- J2 pad 2: unconnected-(J2-Pin_2-Pad2) -> GND
Routing:
- net GND: track 118.2 -> 176.1 mm, vias 4 -> 8
- net Net-(J1-CC1): track 21.9 -> 17.3 mm
- net Net-(U1-VCAP_2): track 13.7 -> 17.1 mm
- net unconnected-(J2-Pin_2-Pad2): track 0.76 -> 0.00 mm
- added copper zone on F.Cu, net /USB_+
- added copper zone on F.Cu, net /USB_-

Commit message: refresh
Routing:
- net GND: track 176.1 -> 179.4 mm, vias 8 -> 10

Commit message: refresh
Parts:
- added U3: W25Q128JVP, Package_SON:WSON-8-1EP_6x5mm_P1.27mm_EP3.4x4.3mm, F.Cu at (171.7, 87.7)
Connections:
- J2 pad 2: GND -> unconnected-(J2-Pin_2-Pad2)
Routing:
- net unconnected-(J2-Pin_2-Pad2): track 0.00 -> 0.76 mm
- net GND: track 179.4 -> 178.6 mm

Commit message: refresh
Parts:
- added C15: C_Polarized, Capacitor_Tantalum_SMD:CP_EIA-6032-28_Kemet-C, F.Cu at (174.4, 80.0)
- added C16: C, Capacitor_SMD:C_1206_3216Metric, F.Cu at (170.6, 81.0)
Connections:
- C10 pad 1: Net-(C10-Pad1) -> Net-(J2-Pin_2)
- C11 pad 1: Net-(C11-Pad1) -> Net-(J2-Pin_2)
- C12 pad 1: Net-(C11-Pad1) -> Net-(J2-Pin_2)
- C13 pad 1: Net-(U1-VDDA) -> Net-(J2-Pin_2)
- C14 pad 1: Net-(U1-VDDA) -> Net-(J2-Pin_2)
- C3 pad 1: Net-(C3-Pad1) -> Net-(J2-Pin_2)
- C4 pad 1: Net-(C3-Pad1) -> Net-(J2-Pin_2)
- C5 pad 1: Net-(C5-Pad1) -> Net-(J2-Pin_2)
- C6 pad 1: Net-(C5-Pad1) -> Net-(J2-Pin_2)
- C7 pad 1: Net-(C7-Pad1) -> Net-(J2-Pin_2)
- C8 pad 1: Net-(C7-Pad1) -> Net-(J2-Pin_2)
- C9 pad 1: Net-(C10-Pad1) -> Net-(J2-Pin_2)
- FB1 pad 1: Net-(C3-Pad1) -> Net-(J2-Pin_2)
- J2 pad 2: unconnected-(J2-Pin_2-Pad2) -> Net-(J2-Pin_2)
- U1 pad 13: Net-(U1-VDDA) -> Net-(J2-Pin_2)
- U1 pad 19: Net-(C5-Pad1) -> Net-(J2-Pin_2)
- U1 pad 20: unconnected-(U1-PA4-Pad20) -> Net-(U1-PA4)
- U1 pad 21: unconnected-(U1-PA5-Pad21) -> Net-(U1-PA5)
- U1 pad 22: unconnected-(U1-PA6-Pad22) -> Net-(U1-PA6)
- U1 pad 23: unconnected-(U1-PA7-Pad23) -> Net-(U1-PA7)
- U1 pad 32: Net-(C7-Pad1) -> Net-(J2-Pin_2)
- U1 pad 48: Net-(C10-Pad1) -> Net-(J2-Pin_2)
- U1 pad 64: Net-(C11-Pad1) -> Net-(J2-Pin_2)
- U3 pad 1: unconnected-(U3-~{CS}-Pad1) -> Net-(U1-PA4)
- U3 pad 2: unconnected-(U3-DO/IO_{1}-Pad2) -> Net-(U1-PA7)
- U3 pad 3: unconnected-(U3-~{WP}/IO_{2}-Pad3) -> Net-(J2-Pin_2)
- U3 pad 4: unconnected-(U3-GND-Pad4) -> GND
- U3 pad 5: unconnected-(U3-DI/IO_{0}-Pad5) -> Net-(U1-PA6)
- U3 pad 6: unconnected-(U3-CLK-Pad6) -> Net-(U1-PA5)
- U3 pad 7: unconnected-(U3-~{HOLD}/~{RESET}/IO_{3}-Pad7) -> Net-(J2-Pin_2)
- U3 pad 8: unconnected-(U3-VCC-Pad8) -> Net-(J2-Pin_2)
- U3 pad 9: unconnected-(U3-EP-Pad9) -> GND
Routing:
- net Net-(J2-Pin_2): track 0.00 -> 80.0 mm, vias 0 -> 8
- net Net-(U1-PA7): track 0.00 -> 30.8 mm, vias 0 -> 2
- net Net-(U1-PA5): track 0.00 -> 22.0 mm, vias 0 -> 2
- net Net-(U1-PA4): track 0.00 -> 21.3 mm, vias 0 -> 2
- net Net-(U1-PA6): track 0.00 -> 20.5 mm, vias 0 -> 2
- net GND: track 178.6 -> 197.7 mm, vias 10 -> 13
- net Net-(U1-VDDA): track 15.6 -> 0.00 mm, vias 1 -> 0
- net Net-(C10-Pad1): track 12.0 -> 0.00 mm, vias 1 -> 0
- net Net-(C3-Pad1): track 10.0 -> 0.00 mm, vias 1 -> 0
- net Net-(C11-Pad1): track 9.31 -> 0.00 mm, vias 1 -> 0
- net Net-(C7-Pad1): track 8.56 -> 0.00 mm, vias 1 -> 0
- net Net-(C5-Pad1): track 8.56 -> 0.00 mm, vias 1 -> 0
- net unconnected-(J2-Pin_2-Pad2): track 0.76 -> 0.00 mm
- added copper zone on In2.Cu, net Net-(J2-Pin_2)
- removed copper zone on In2.Cu, net unconnected-(J2-Pin_2-Pad2)

Commit message: refresh
Routing:
- net Net-(J2-Pin_2): track 80.0 -> 85.7 mm
