File: microcontroller/micro/micro.kicad_pcb (KiCad board)
At the start: 4 copper layers, 60 x 60 mm, 25 parts, among them J1 USB_C_Receptacle_USB2.0_16P, U1 STM32F405RGTx, U2 TPD4E05U06DQA, U3 W25Q128JVP, U4 SX1276

Commit message: refresh
Parts:
- added J2: Screw_Terminal_01x10, Connector_PinHeader_2.54mm:PinHeader_1x10_P2.54mm_Vertical, F.Cu at (156.1, 74.0)
Connections:
- U1 pad 26: unconnected-(U1-PB0-Pad26) -> /1-1
- U1 pad 28: unconnected-(U1-PB2-Pad28) -> /1-2
- U1 pad 29: unconnected-(U1-PB10-Pad29) -> /1-6
- U1 pad 30: unconnected-(U1-PB11-Pad30) -> /1-7
- U1 pad 33: unconnected-(U1-PB12-Pad33) -> /1-8
- U1 pad 34: unconnected-(U1-PB13-Pad34) -> /1-9
- U1 pad 35: unconnected-(U1-PB14-Pad35) -> /1-10
- U1 pad 57: unconnected-(U1-PB5-Pad57) -> /1-3
- U1 pad 61: unconnected-(U1-PB8-Pad61) -> /1-4
- U1 pad 62: unconnected-(U1-PB9-Pad62) -> /1-5
Routing:
- net /1-2: track 0.00 -> 39.2 mm
- net /1-1: track 0.00 -> 38.0 mm
- net /1-3: track 0.00 -> 32.5 mm
Other:
- copper layers 4 -> 6
- rule pad_to_mask_clearance: 0 -> 0.03

Commit message: refresh
Routing:
- net /1-2: track 39.2 -> 0.00 mm
- net /1-1: track 38.0 -> 0.00 mm
- net Net-(U1-PB3): track 36.6 -> 0.00 mm, vias 1 -> 0
- net Net-(U1-PB4): track 36.6 -> 0.00 mm, vias 1 -> 0
- net Net-(U1-PB1): track 36.4 -> 0.00 mm, vias 1 -> 0
- net /1-3: track 32.5 -> 0.00 mm
- net Net-(U1-PB6): track 30.6 -> 0.00 mm, vias 1 -> 0
- net Net-(U1-PB7): track 30.6 -> 0.00 mm, vias 1 -> 0
- net Net-(U1-PA7): track 30.8 -> 19.5 mm
- net Net-(U1-PA4): track 30.9 -> 21.3 mm
- net Net-(U1-VDDA): track 82.6 -> 89.8 mm, vias 9 -> 8
- net Net-(U1-PA6): track 30.6 -> 25.9 mm
- net Net-(U1-PA5): track 30.9 -> 28.6 mm

Commit message: length tuning
Routing:
- net Net-(U1-PA7): track 19.5 -> 28.5 mm
- net Net-(U1-PA4): track 21.3 -> 28.5 mm
- net Net-(U1-PA6): track 25.9 -> 28.5 mm

Commit message: refresh
Routing:
- net /1-1: track 0.00 -> 40.4 mm, vias 0 -> 1
- net Net-(U1-PB6): track 0.00 -> 38.5 mm, vias 0 -> 1
- net Net-(U1-PB4): track 0.00 -> 36.2 mm, vias 0 -> 1
- net Net-(U1-PB3): track 0.00 -> 35.9 mm, vias 0 -> 1
- net /1-2: track 0.00 -> 35.5 mm, vias 0 -> 1
- net Net-(U1-PB1): track 0.00 -> 34.9 mm, vias 0 -> 1
- net /1-7: track 0.00 -> 32.2 mm, vias 0 -> 1
- net /1-6: track 0.00 -> 31.6 mm, vias 0 -> 1
- net unconnected-(U1-PC4-Pad24): track 0.00 -> 1.34 mm, vias 0 -> 1
- net /1-3: track 0.00 -> 1.31 mm, vias 0 -> 1
- removed copper zone on In1.Cu, net GND
- removed copper zone on In2.Cu, net Net-(U1-VDDA)

Commit message: refresh
Routing:
- net /1-8: track 0.00 -> 40.8 mm, vias 0 -> 1
- net /1-4: track 0.00 -> 40.5 mm
- net /1-9: track 0.00 -> 39.9 mm, vias 0 -> 1
- net /1-5: track 0.00 -> 39.8 mm
- net /1-10: track 0.00 -> 39.8 mm, vias 0 -> 1
- net /1-3: track 1.31 -> 40.1 mm, vias 1 -> 0
- net Net-(U1-PB7): track 0.00 -> 34.7 mm, vias 0 -> 1
- net /1-6: track 31.6 -> 40.5 mm
- net /1-7: track 32.2 -> 39.6 mm
- net /1-2: track 35.5 -> 40.6 mm
- added copper zone on B.Cu, net GND
- added copper zone on F.Cu, net GND
- added copper zone on In1.Cu, net GND
- added copper zone on In2.Cu, net GND
- added copper zone on In4.Cu, net GND
- added copper zone on In3.Cu, net Net-(U1-VDDA)

Commit message: refresh
Routing:
- removed copper zone on B.Cu, net GND
- removed copper zone on F.Cu, net GND
- removed copper zone on In1.Cu, net GND
- removed copper zone on In2.Cu, net GND
- removed copper zone on In4.Cu, net GND
- removed copper zone on In3.Cu, net Net-(U1-VDDA)

Commit message: refresh
Parts:
- added J3: Screw_Terminal_01x02, Connector_PinHeader_2.54mm:PinHeader_1x02_P2.54mm_Vertical, B.Cu at (148.0, 80.3)
- added J4: Screw_Terminal_01x02, Connector_PinHeader_2.54mm:PinHeader_1x02_P2.54mm_Vertical, B.Cu at (187.8, 81.1)
- added J5: Screw_Terminal_01x02, Connector_PinHeader_2.54mm:PinHeader_1x02_P2.54mm_Vertical, B.Cu at (146.6, 114.7)
- added J6: Screw_Terminal_01x02, Connector_PinHeader_2.54mm:PinHeader_1x02_P2.54mm_Vertical, B.Cu at (188.4, 114.7)
Connections:
- net Net-(U1-VDDA) renamed +3.3V
Routing:
- net Net-(U1-PB4): track 36.2 -> 43.4 mm
- net Net-(U1-PB7): track 34.7 -> 41.3 mm
- net Net-(U1-PB6): track 38.5 -> 43.1 mm

Commit message: refresh
Parts:
- added J10: Screw_Terminal_01x02, Connector_PinHeader_2.54mm:PinHeader_1x02_P2.54mm_Vertical, F.Cu at (184.5, 79.0)
- added J7: Screw_Terminal_01x02, Connector_PinHeader_2.54mm:PinHeader_1x02_P2.54mm_Vertical, F.Cu at (184.5, 113.0)
- added J8: Screw_Terminal_01x02, Connector_PinHeader_2.54mm:PinHeader_1x02_P2.54mm_Vertical, F.Cu at (150.5, 113.0)
- added J9: Screw_Terminal_01x02, Connector_PinHeader_2.54mm:PinHeader_1x02_P2.54mm_Vertical, F.Cu at (150.5, 79.0)
- moved J3 36.3 mm to (150.5, 116.5)
- moved J4 35.5 mm to (184.5, 116.5)
- moved J5 32.5 mm to (150.5, 82.5)
- moved J6 32.5 mm to (184.5, 82.5)
Routing:
- net Net-(U1-PB4): track 43.4 -> 35.1 mm
- net Net-(U1-PB6): track 43.1 -> 38.5 mm
- net Net-(U1-PB3): track 35.9 -> 35.1 mm
