File: microcontroller/micro/micro.kicad_sch (KiCad schematic)
At the start: 16 parts, among them U1 STM32F405RGTx

Commit message: refresh
Parts:
- added J1: USB_C_Receptacle_USB2.0_16P, Connector_USB:USB_C_Receptacle_GCT_USB4105-xx-A_16P_TopMnt_Horizontal, symbol Connector:USB_C_Receptacle_USB2.0_16P
- added R1, R2: 5.1k, Resistor_SMD:R_01005_0402Metric, symbol Device:R_US
- added R3: 4.7k, Resistor_SMD:R_01005_0402Metric, symbol Device:R_US
- added U2: TPD4E05U06DQA, Package_SON:USON-10_2.5x1.0mm_P0.5mm, symbol Power_Protection:TPD4E05U06DQA
Connections:
- net GND: now also J1.A1 (GND), J1.A12 (GND), J1.B1 (GND), J1.B12 (GND), J1.SH (SHIELD), R1.1, R2.1, U2.3 (GND), U2.8 (GND)
- net at U1.42 (PA9): now also R3.1
- net USB_-: now reaches U1.44 (PA11)
- net USB_-: now also J1.A7 (D-), U2.2 (D1-)
- net USB_+: now reaches U1.45 (PA12)
- net USB_+: now also J1.B6 (D+), U2.1 (D1+)
- new net: J1.B5 (CC2), R1.2, U2.4 (D2+)
- new net: J1.A5 (CC1), R2.2, U2.5 (D2-)
- new net: J1.A4 (VBUS), J1.A9 (VBUS), J1.B4 (VBUS), J1.B9 (VBUS), R3.2
Other:
- moved on the sheet: C10, C11, C12, C13, C14, C3, C4, C5, C6, C7, C8, C9

Commit message: refresh
Parts:
- C1, C10, C12, C14, C2, C3, C6, C8: footprint Capacitor_SMD:C_01005_0402Metric -> Capacitor_SMD:C_1206_3216Metric
- R1, R2: footprint Resistor_SMD:R_01005_0402Metric -> Resistor_SMD:R_1206_3216Metric
- R3: footprint Resistor_SMD:R_01005_0402Metric -> Resistor_SMD:R_0603_1608Metric
Connections:
- net USB_+: now also U2.10 (NC)
- net USB_-: now also U2.9 (NC)
- net at J1.B5 (CC2), R1.2, U2.4 (D2+): now also U2.7 (NC)
- net at J1.A5 (CC1), R2.2, U2.5 (D2-): now also U2.6 (NC)
Changed lines of the file:
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@@
+	)
+	(junction
+		(at 207.01 50.8)
+		(diameter 0)
+		(color 0 0 0 0)
 	)
 	(junction
@@
 	)
 	(junction
+		(at 181.61 45.72)
+		(diameter 0)
+		(color 0 0 0 0)
+	)
+	(junction
 		(at 120.65 39.37)
 		(diameter 0)
@@
 	)
 	(junction
+		(at 181.61 50.8)
+		(diameter 0)
+		(color 0 0 0 0)
+	)
+	(junction
 		(at 143.51 146.05)
 		(diameter 0)
@@
 	)
 	(junction
-		(at 208.28 74.93)
-		(diameter 0)
-		(color 0 0 0 0)
-	)
-	(junction
 		(at 148.59 39.37)
 		(diameter 0)
@@
 	)
 	(junction
-		(at 210.82 77.47)
+		(at 156.21 31.75)
 		(diameter 0)
 		(color 0 0 0 0)
 	)
 	(junction
-		(at 156.21 31.75)
+		(at 207.01 45.72)
 		(diameter 0)
 		(color 0 0 0 0)
@@
 	)
 	(junction
+		(at 212.09 77.47)
+		(diameter 0)
+		(color 0 0 0 0)
+	)
+	(junction
 		(at 135.89 39.37)
 		(diameter 0)
@@
 		(color 0 0 0 0)
 	)
+	(junction
+		(at 209.55 74.93)
+		(diameter 0)
+		(color 0 0 0 0)
+	)
 	(wire
 		(pts
@@
 	(wire
 		(pts
+			(xy 181.61 50.8) (xy 181.61 55.88)
+		)
+		(stroke
+			(width 0)
+			(type default)
+		)
+	)
+	(wire
+		(pts
 			(xy 149.86 45.72) (xy 149.86 49.53)
 		)
@@
 	(wire
 		(pts
-			(xy 204.47 74.93) (xy 208.28 74.93)
+			(xy 204.47 74.93) (xy 209.55 74.93)
 		)
 		(stroke
@@
 	(wire
 		(pts
-			(xy 207.01 50.8) (xy 208.28 50.8)
+			(xy 207.01 50.8) (xy 209.55 50.8)
 		)
 		(stroke
@@
 	(wire
 		(pts
-			(xy 210.82 77.47) (xy 226.06 77.47)
-		)
-		(stroke
-			(width 0)
-			(type default)
-		)
-	)
-	(wire
-		(pts
 			(xy 196.85 74.93) (xy 196.85 76.2)
 		)
@@
 	(wire
 		(pts
-			(xy 208.28 50.8) (xy 208.28 74.93)
+			(xy 209.55 50.8) (xy 209.55 74.93)
+		)
+		(stroke
+			(width 0)
+			(type default)
+		)
+	)
+	(wire
+		(pts
+			(xy 209.55 74.93) (xy 226.06 74.93)
 		)
 		(stroke
@@
 	(wire
 		(pts
+			(xy 207.01 50.8) (xy 207.01 55.88)
+		)
+		(stroke
+			(width 0)
+			(type default)
+		)
+	)
+	(wire
+		(pts
 			(xy 120.65 31.75) (xy 125.73 31.75)
 		)
@@
 	(wire
 		(pts
+			(xy 207.01 40.64) (xy 207.01 45.72)
+		)
+		(stroke
+			(width 0)
+			(type default)
+		)
+	)
+	(wire
+		(pts
 			(xy 158.75 39.37) (xy 153.67 44.45)
 		)
@@
 	(wire
 		(pts
+			(xy 212.09 77.47) (xy 226.06 77.47)
+		)
+		(stroke
+			(width 0)
+			(type default)
+		)
+	)
+	(wire
+		(pts
 			(xy 142.24 43.18) (xy 142.24 49.53)
 		)
@@
 	(wire
 		(pts
-			(xy 208.28 74.93) (xy 226.06 74.93)
-		)
-		(stroke
-			(width 0)
-			(type default)
-		)
-	)
-	(wire
-		(pts
-			(xy 207.01 45.72) (xy 210.82 45.72)
+			(xy 181.61 40.64) (xy 181.61 45.72)
+		)
+		(stroke
+			(width 0)
+			(type default)
+		)
+	)
+	(wire
+		(pts
+			(xy 207.01 45.72) (xy 212.09 45.72)
 		)
 		(stroke
@@
 	(wire
 		(pts
-			(xy 204.47 77.47) (xy 210.82 77.47)
+			(xy 204.47 77.47) (xy 212.09 77.47)
 		)
 		(stroke
@@
 	(wire
 		(pts
-			(xy 210.82 45.72) (xy 210.82 77.47)
+			(xy 212.09 45.72) (xy 212.09 77.47)
 		)
 		(stroke
@@
 			)
 		)
-		(property "Footprint" "Capacitor_SMD:C_01005_0402Metric"
+		(property "Footprint" "Capacitor_SMD:C_1206_3216Metric"
 			(at 105.1052 134.62 0)
 			(hide yes)
@@
 			)
 		)
-		(property "Footprint" "Capacitor_SMD:C_01005_0402Metric"
+		(property "Footprint" "Capacitor_SMD:C_1206_3216Metric"
 			(at 117.8052 134.62 0)
 			(hide yes)
@@
 			)
 		)
-		(property "Footprint" "Capacitor_SMD:C_01005_0402Metric"
+		(property "Footprint" "Capacitor_SMD:C_1206_3216Metric"
 			(at 170.4848 31.75 0)
 			(hide yes)
@@
 			)
 		)
-		(property "Footprint" "Resistor_SMD:R_01005_0402Metric"
+		(property "Footprint" "Resistor_SMD:R_1206_3216Metric"
 			(at 200.914 76.454 90)
 			(hide yes)
@@
 			)
 		)
-		(property "Footprint" "Capacitor_SMD:C_01005_0402Metric"
+		(property "Footprint" "Capacitor_SMD:C_1206_3216Metric"
 			(at 150.1648 31.75 0)
 			(hide yes)
@@
 			)
 		)
-		(property "Footprint" "Capacitor_SMD:C_01005_0402Metric"
+		(property "Footprint" "Capacitor_SMD:C_1206_3216Metric"
 			(at 119.6848 31.75 0)
 			(hide yes)
@@
 			)
 		)
-		(property "Footprint" "Resistor_SMD:R_01005_0402Metric"
+		(property "Footprint" "Resistor_SMD:R_0603_1608Metric"
 			(at 200.914 68.834 90)
 			(hide yes)
@@
 			)
 		)
-		(property "Footprint" "Capacitor_SMD:C_01005_0402Metric"
+		(property "Footprint" "Capacitor_SMD:C_1206_3216Metric"
 			(at 129.8448 31.75 0)
 			(hide yes)
@@
 			)
 		)
-		(property "Footprint" "Capacitor_SMD:C_01005_0402Metric"
+		(property "Footprint" "Capacitor_SMD:C_1206_3216Metric"
 			(at 160.3248 31.75 0)
 			(hide yes)
@@
 			)
 		)
-		(property "Footprint" "Resistor_SMD:R_01005_0402Metric"
+		(property "Footprint" "Resistor_SMD:R_1206_3216Metric"
 			(at 200.914 73.914 90)
 			(hide yes)
@@
 			)
 		)
-		(property "Footprint" "Capacitor_SMD:C_01005_0402Metric"
+		(property "Footprint" "Capacitor_SMD:C_1206_3216Metric"
 			(at 140.0048 31.75 0)
 			(hide yes)

Commit message: refresh
Parts:
- added J2: Screw_Terminal_01x03, Connector_JST:JST_EH_B3B-EH-A_1x03_P2.50mm_Vertical, symbol Connector:Screw_Terminal_01x03
Connections:
- net GND: now also J2.1 (Pin_1)
- net at C10.1, C11.1, C12.1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: now also J2.2 (Pin_2)
- no-connect marks 0 -> 1
Changed lines of the file:
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@@
+	)
+	(junction
+		(at 115.57 39.37)
+		(diameter 0)
+		(color 0 0 0 0)
 	)
 	(junction
@@
 		(color 0 0 0 0)
 	)
+	(no_connect
+		(at 48.26 76.2)
+	)
 	(wire
 		(pts
@@
 	(wire
 		(pts
+			(xy 48.26 78.74) (xy 76.2 78.74)
+		)
+		(stroke
+			(width 0)
+			(type default)
+		)
+	)
+	(wire
+		(pts
 			(xy 226.06 82.55) (xy 222.25 82.55)
 		)
@@
 	(wire
 		(pts
+			(xy 76.2 78.74) (xy 115.57 39.37)
+		)
+		(stroke
+			(width 0)
+			(type default)
+		)
+	)
+	(wire
+		(pts
 			(xy 135.89 31.75) (xy 140.97 31.75)
 		)
@@
 		(pts
 			(xy 179.07 50.8) (xy 179.07 85.09)
+		)
+		(stroke
+			(width 0)
+			(type default)
+		)
+	)
+	(wire
+		(pts
+			(xy 50.8 81.28) (xy 48.26 81.28)
 		)
 		(stroke
@@
 	)
 	(symbol
+		(lib_id "Connector:Screw_Terminal_01x03")
+		(at 43.18 78.74 180)
+		(unit 1)
+		(body_style 1)
+		(exclude_from_sim no)
+		(in_bom yes)
+		(on_board yes)
+		(in_pos_files yes)
+		(dnp no)
+		(fields_autoplaced yes)
+		(property "Reference" "J2"
+			(at 43.18 72.39 0)
+			(show_name no)
+			(do_not_autoplace no)
+			(effects
+				(font
+					(size 1.27 1.27)
+				)
+			)
+		)
+		(property "Value" "Screw_Terminal_01x03"
+			(at 40.64 77.4701 0)
+			(hide yes)
+			(show_name no)
+			(do_not_autoplace no)
+			(effects
+				(font
+					(size 1.27 1.27)
+				)
+				(justify left)
+			)
+		)
+		(property "Footprint" "Connector_JST:JST_EH_B3B-EH-A_1x03_P2.50mm_Vertical"
+			(at 43.18 78.74 0)
+			(hide yes)
+			(show_name no)
+			(do_not_autoplace no)
+			(effects
+				(font
+					(size 1.27 1.27)
+				)
+			)
+		)
+		(property "Datasheet" ""
+			(at 43.18 78.74 0)
+			(hide yes)
+			(show_name no)
+			(do_not_autoplace no)
+			(effects
+				(font
+					(size 1.27 1.27)
+				)
+			)
+		)
+		(property "Description" "Generic screw terminal, single row, 01x03, script generated (kicad-library-utils/schlib/autogen/connector/)"
+			(at 43.18 78.74 0)
+			(hide yes)
+			(show_name no)
+			(do_not_autoplace no)
+			(effects
+				(font
+					(size 1.27 1.27)
+				)
+			)
+		)
+		(pin "1"
+		)
+		(pin "2"
+		)
+		(pin "3"
+		)
+		(instances
+			(project "micro"
+				(path "/20867279-5aff-4560-94cd-e855d560edf3"
+					(reference "J2")
+					(unit 1)
+				)
+			)
+		)
+	)
+	(symbol
 		(lib_id "MCU_ST_STM32F4:STM32F405RGTx")
 		(at 142.24 97.79 0)
@@
 					(unit 1)
 				)
+			)
+		)
+	)
+	(symbol
+		(lib_id "power:GND")
+		(at 50.8 81.28 0)
+		(unit 1)
+		(body_style 1)
+		(exclude_from_sim no)
+		(in_bom yes)
+		(on_board yes)
+		(in_pos_files yes)
+		(dnp no)
+		(fields_autoplaced yes)
+		(property "Reference" "#PWR08"
+			(at 50.8 87.63 0)
+			(hide yes)
+			(show_name no)
+			(do_not_autoplace no)
+			(effects
+				(font
+					(size 1.27 1.27)
+				)
+			)
+		)
+		(property "Value" "GND"
+			(at 50.8 86.36 0)
+			(show_name no)
+			(do_not_autoplace no)
+			(effects
+				(font
+					(size 1.27 1.27)
+				)
+			)
+		)
+		(property "Footprint" ""
+			(at 50.8 81.28 0)
+			(hide yes)
+			(show_name no)
+			(do_not_autoplace no)
+			(effects
+				(font
+					(size 1.27 1.27)
+				)
+			)
+		)
+		(property "Datasheet" ""
+			(at 50.8 81.28 0)
+			(hide yes)
+			(show_name no)
+			(do_not_autoplace no)
+			(effects
+				(font
+					(size 1.27 1.27)
+				)
+			)
+		)
+		(property "Description" "Power symbol creates a global label with name \"GND\" , ground"
+			(at 50.8 81.28 0)
+			(hide yes)
+			(show_name no)
+			(do_not_autoplace no)
+			(effects
+				(font
+					(size 1.27 1.27)
+				)
+			)
+		)
+		(pin "1"
+		)
+		(instances
+			(project "micro"
+				(path "/20867279-5aff-4560-94cd-e855d560edf3"
+					(reference "#PWR08")
+					(unit 1)
+				)

Commit message: refresh
Parts:
- C11, C13, C4, C5, C7, C9: footprint Capacitor_Tantalum_SMD:CP_EIA-1608-08_AVX-J -> Capacitor_Tantalum_SMD:CP_EIA-6032-28_Kemet-C
- FB1: footprint Ferrite_THT:LairdTech_28C0236-0JW-10 -> Inductor_SMD:L_Walsin_WLFM201609x
Connections:
- new net: C13.1, C14.1, U1.13 (VDDA)
- new net: C11.1, C12.1, U1.64 (VDD)
- new net: C7.1, C8.1, U1.32 (VDD)
- new net: C10.1, C9.1, U1.48 (VDD)
- new net: C3.1, C4.1, FB1.1
- new net: C5.1, C6.1, U1.19 (VDD)
- now unconnected: J2.2 (Pin_2)
Changed lines of the file:
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@@
 	)
 	(junction
-		(at 166.37 39.37)
-		(diameter 0)
-		(color 0 0 0 0)
-	)
-	(junction
 		(at 128.27 39.37)
 		(diameter 0)
@@
 	)
 	(junction
-		(at 130.81 39.37)
-		(diameter 0)
-		(color 0 0 0 0)
-	)
-	(junction
 		(at 130.81 31.75)
 		(diameter 0)
@@
 	)
 	(junction
-		(at 140.97 39.37)
-		(diameter 0)
-		(color 0 0 0 0)
-	)
-	(junction
-		(at 125.73 39.37)
-		(diameter 0)
-		(color 0 0 0 0)
-	)
-	(junction
 		(at 118.11 39.37)
 		(diameter 0)
@@
 	)
 	(junction
-		(at 120.65 39.37)
-		(diameter 0)
-		(color 0 0 0 0)
-	)
-	(junction
-		(at 146.05 39.37)
-		(diameter 0)
-		(color 0 0 0 0)
-	)
-	(junction
 		(at 181.61 50.8)
 		(diameter 0)
@@
 	)
 	(junction
-		(at 156.21 39.37)
-		(diameter 0)
-		(color 0 0 0 0)
-	)
-	(junction
-		(at 151.13 39.37)
-		(diameter 0)
-		(color 0 0 0 0)
-	)
-	(junction
 		(at 161.29 31.75)
 		(diameter 0)
@@
 	)
 	(junction
-		(at 115.57 39.37)
-		(diameter 0)
-		(color 0 0 0 0)
-	)
-	(junction
 		(at 156.21 31.75)
 		(diameter 0)
@@
 	)
 	(junction
-		(at 135.89 39.37)
-		(diameter 0)
-		(color 0 0 0 0)
-	)
-	(junction
 		(at 135.89 31.75)
 		(diameter 0)
@@
 	)
 	(junction
-		(at 161.29 39.37)
-		(diameter 0)
-		(color 0 0 0 0)
-	)
-	(junction
 		(at 209.55 74.93)
 		(diameter 0)
@@
 	(wire
 		(pts
-			(xy 151.13 39.37) (xy 156.21 39.37)
-		)
-		(stroke
-			(width 0)
-			(type default)
-		)
-	)
-	(wire
-		(pts
 			(xy 181.61 50.8) (xy 181.61 55.88)
 		)
@@
 	(wire
 		(pts
-			(xy 130.81 39.37) (xy 135.89 39.37)
-		)
-		(stroke
-			(width 0)
-			(type default)
-		)
-	)
-	(wire
-		(pts
 			(xy 118.11 39.37) (xy 120.65 39.37)
 		)
@@
 	(wire
 		(pts
-			(xy 76.2 78.74) (xy 115.57 39.37)
-		)
-		(stroke
-			(width 0)
-			(type default)
-		)
-	)
-	(wire
-		(pts
 			(xy 135.89 31.75) (xy 140.97 31.75)
 		)
@@
 	(wire
 		(pts
-			(xy 161.29 39.37) (xy 166.37 39.37)
-		)
-		(stroke
-			(width 0)
-			(type default)
-		)
-	)
-	(wire
-		(pts
 			(xy 168.91 39.37) (xy 171.45 39.37)
 		)
@@
 	(wire
 		(pts
-			(xy 140.97 39.37) (xy 146.05 39.37)
-		)
-		(stroke
-			(width 0)
-			(type default)
-		)
-	)
-	(wire
-		(pts
 			(xy 207.01 50.8) (xy 207.01 55.88)
 		)
@@
 	(wire
 		(pts
-			(xy 120.65 39.37) (xy 125.73 39.37)
-		)
-		(stroke
-			(width 0)
-			(type default)
-		)
-	)
-	(wire
-		(pts
 			(xy 196.85 76.2) (xy 196.85 77.47)
 		)
@@
 			)
 		)
-		(property "Footprint" "Capacitor_Tantalum_SMD:CP_EIA-1608-08_AVX-J"
+		(property "Footprint" "Capacitor_Tantalum_SMD:CP_EIA-6032-28_Kemet-C"
 			(at 155.2448 31.75 0)
 			(hide yes)
@@
 			)
 		)
-		(property "Footprint" "Capacitor_Tantalum_SMD:CP_EIA-1608-08_AVX-J"
+		(property "Footprint" "Capacitor_Tantalum_SMD:CP_EIA-6032-28_Kemet-C"
 			(at 134.9248 31.75 0)
 			(hide yes)
@@
 			)
 		)
-		(property "Footprint" "Capacitor_Tantalum_SMD:CP_EIA-1608-08_AVX-J"
+		(property "Footprint" "Capacitor_Tantalum_SMD:CP_EIA-6032-28_Kemet-C"
 			(at 124.7648 31.75 0)
 			(hide yes)
@@
 			)
 		)
-		(property "Footprint" "Ferrite_THT:LairdTech_28C0236-0JW-10"
+		(property "Footprint" "Inductor_SMD:L_Walsin_WLFM201609x"
 			(at 128.27 47.498 90)
 			(hide yes)
@@
 			)
 		)
-		(property "Footprint" "Capacitor_Tantalum_SMD:CP_EIA-1608-08_AVX-J"
+		(property "Footprint" "Capacitor_Tantalum_SMD:CP_EIA-6032-28_Kemet-C"
 			(at 165.4048 31.75 0)
 			(hide yes)
@@
 			)
 		)
-		(property "Footprint" "Capacitor_Tantalum_SMD:CP_EIA-1608-08_AVX-J"
+		(property "Footprint" "Capacitor_Tantalum_SMD:CP_EIA-6032-28_Kemet-C"
 			(at 145.0848 31.75 0)
 			(hide yes)
@@
 			)
 		)
-		(property "Footprint" "Capacitor_Tantalum_SMD:CP_EIA-1608-08_AVX-J"
+		(property "Footprint" "Capacitor_Tantalum_SMD:CP_EIA-6032-28_Kemet-C"
 			(at 114.6048 31.75 0)
 			(hide yes)

Commit message: refresh
Parts:
- added U3: W25Q128JVP, Package_SON:WSON-8-1EP_6x5mm_P1.27mm_EP3.4x4.3mm, symbol Memory_Flash:W25Q128JVP
Changed lines of the file:
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@@
+	)
+	(symbol
+		(lib_id "Memory_Flash:W25Q128JVP")
+		(at 58.42 113.03 0)
+		(unit 1)
+		(body_style 1)
+		(exclude_from_sim no)
+		(in_bom yes)
+		(on_board yes)
+		(in_pos_files yes)
+		(dnp no)
+		(fields_autoplaced yes)
+		(property "Reference" "U3"
+			(at 69.85 111.7599 0)
+			(show_name no)
+			(do_not_autoplace no)
+			(effects
+				(font
+					(size 1.27 1.27)
+				)
+				(justify left)
+			)
+		)
+		(property "Value" "W25Q128JVP"
+			(at 69.85 114.2999 0)
+			(show_name no)
+			(do_not_autoplace no)
+			(effects
+				(font
+					(size 1.27 1.27)
+				)
+				(justify left)
+			)
+		)
+		(property "Footprint" "Package_SON:WSON-8-1EP_6x5mm_P1.27mm_EP3.4x4.3mm"
+			(at 58.42 90.17 0)
+			(hide yes)
+			(show_name no)
+			(do_not_autoplace no)
+			(effects
+				(font
+					(size 1.27 1.27)
+				)
+			)
+		)
+		(property "Datasheet" "https://www.winbond.com/resource-files/w25q128jv_dtr%20revc%2003272018%20plus.pdf"
+			(at 58.42 87.63 0)
+			(hide yes)
+			(show_name no)
+			(do_not_autoplace no)
+			(effects
+				(font
+					(size 1.27 1.27)
+				)
+			)
+		)
+		(property "Description" "128Mbit / 16MiB Serial Flash Memory, Standard/Dual/Quad SPI, 2.7-3.6V, WSON-8"
+			(at 58.42 85.09 0)
+			(hide yes)
+			(show_name no)
+			(do_not_autoplace no)
+			(effects
+				(font
+					(size 1.27 1.27)
+				)
+			)
+		)
+		(pin "5"
+		)
+		(pin "4"
+		)
+		(pin "6"
+		)
+		(pin "3"
+		)
+		(pin "1"
+		)
+		(pin "7"
+		)
+		(pin "8"
+		)
+		(pin "9"
+		)
+		(pin "2"
+		)
+		(instances
+			(project "micro"
+				(path "/20867279-5aff-4560-94cd-e855d560edf3"
+					(reference "U3")
+					(unit 1)
+				)
+			)
+		)
 	)
 	(symbol

Commit message: refresh
Parts:
- added C15: C_Polarized, Capacitor_Tantalum_SMD:CP_EIA-6032-28_Kemet-C, symbol Device:C_Polarized
- added C16: C, Capacitor_SMD:C_1206_3216Metric, symbol Device:C
Connections:
- net GND: now also U3.4 (GND), U3.9 (EP), C15.2, C16.2
- net at C13.1, C14.1, U1.13 (VDDA): now also C10.1, C11.1, C12.1, C3.1, C4.1, C5.1, C6.1, C7.1, C8.1, C9.1, FB1.1, J2.2 (Pin_2), U1.19 (VDD), U1.32 (VDD), U1.48 (VDD), U1.64 (VDD), U3.3 (~{WP}/IO_{2}), U3.7 (~{HOLD}/~{RESET}/IO_{3}), U3.8 (VCC), C15.1, C16.1
- net at U3.1 (~{CS}): now also U1.20 (PA4)
- net at U3.2 (DO/IO_{1}): now also U1.23 (PA7)
- net at U3.5 (DI/IO_{0}): now also U1.22 (PA6)
- net at U3.6 (CLK): now also U1.21 (PA5)
Other:
- moved on the sheet: U3

Commit message: refresh
Parts:
- removed J2: Screw_Terminal_01x03, Connector_JST:JST_EH_B3B-EH-A_1x03_P2.50mm_Vertical, symbol Connector:Screw_Terminal_01x03
- added U4: SX1276, Connector_PinHeader_2.54mm:PinHeader_1x07_P2.54mm_Vertical, symbol me:SX1276-module
Connections:
- net GND: now also U4.2 (GND)
- net at C10.1, C11.1, C12.1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: now also U4.1 (VCC); no longer C15.1, C16.1, U3.3 (~{WP}/IO_{2}), U3.7 (~{HOLD}/~{RESET}/IO_{3})
- net at U1.27 (PB1): now also U4.5 (AUX)
- net at U1.55 (PB3): now also U4.6 (M0)
- net at U1.56 (PB4): now also U4.7 (M1)
- net at U1.58 (PB6): now also U4.3 (RXD)
- net at U1.59 (PB7): now also U4.4 (TXD)
- new net: C15.1, C16.1, U3.3 (~{WP}/IO_{2}), U3.7 (~{HOLD}/~{RESET}/IO_{3})
- no-connect marks 1 -> 0
Other:
- moved on the sheet: C1, C10, C11, C12, C13, C14, C15, C16, C2, C3, C4, C5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

Commit message: refresh
Connections:
- net at C10.1, C11.1, C12.1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: now also C15.1, C16.1, U3.3 (~{WP}/IO_{2}), U3.7 (~{HOLD}/~{RESET}/IO_{3})
Changed lines of the file:
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@@
+	)
+	(junction
+		(at 139.7 118.11)
+		(diameter 0)
+		(color 0 0 0 0)
 	)
 	(junction
@@
 	)
 	(junction
+		(at 129.54 118.11)
+		(diameter 0)
+		(color 0 0 0 0)
+	)
+	(junction
 		(at 209.55 66.04)
 		(diameter 0)
@@
 		)
 		(stroke
+			(width 0)
+			(type default)
+		)
+	)
+	(wire
+		(pts
+			(xy 129.54 118.11) (xy 139.7 118.11)
+		)
+		(stroke
