File: microcontroller/micro/micro.kicad_sch (KiCad schematic)
At the start: 25 parts, among them J1 USB_C_Receptacle_USB2.0_16P, U1 STM32F405RGTx, U2 TPD4E05U06DQA, U3 W25Q128JVP, U4 SX1276

Commit message: refresh
Parts:
- added J2: Screw_Terminal_01x10, Connector_PinHeader_2.54mm:PinHeader_1x10_P2.54mm_Vertical, symbol Connector:Screw_Terminal_01x10
Connections:
- net 1-1: now reaches U1.26 (PB0)
- net 1-1: now also J2.1 (Pin_1)
- net 1-2: now reaches U1.28 (PB2)
- net 1-2: now also J2.2 (Pin_2)
- net 1-6: now reaches U1.29 (PB10)
- net 1-6: now also J2.6 (Pin_6)
- net 1-7: now reaches U1.30 (PB11)
- net 1-7: now also J2.7 (Pin_7)
- net 1-8: now reaches U1.33 (PB12)
- net 1-8: now also J2.8 (Pin_8)
- net 1-9: now reaches U1.34 (PB13)
- net 1-9: now also J2.9 (Pin_9)
- net 1-10: now reaches U1.35 (PB14)
- net 1-10: now also J2.10 (Pin_10)
- net 1-3: now reaches U1.57 (PB5)
- net 1-3: now also J2.3 (Pin_3)
- net 1-4: now reaches U1.61 (PB8)
- net 1-4: now also J2.4 (Pin_4)
- net 1-5: now reaches U1.62 (PB9)
- net 1-5: now also J2.5 (Pin_5)

Commit message: refresh
Parts:
- added J3, J4, J5, J6: Screw_Terminal_01x02, Connector_PinHeader_2.54mm:PinHeader_1x02_P2.54mm_Vertical, symbol Connector:Screw_Terminal_01x02
Connections:
- net GND: now also J3.1 (Pin_1), J4.1 (Pin_1), J5.1 (Pin_1), J6.1 (Pin_1)
- net +3.3V: now reaches C10.1, C11.1, C12.1, C13.1, C14.1, C15.1, C16.1, C3.1, C4.1, C5.1, C6.1, C7.1, C8.1, C9.1, FB1.1, U1.13 (VDDA), U1.19 (VDD), U1.32 (VDD), U1.48 (VDD), U1.64 (VDD), U3.3 (~{WP}/IO_{2}), U3.7 (~{HOLD}/~{RESET}/IO_{3}), U3.8 (VCC), U4.1 (VCC)
- net +3.3V: now also J3.2 (Pin_2), J4.2 (Pin_2), J5.2 (Pin_2), J6.2 (Pin_2)
Other:
- moved on the sheet: J2

Commit message: refresh
Parts:
- added J10, J7, J8, J9: Screw_Terminal_01x02, Connector_PinHeader_2.54mm:PinHeader_1x02_P2.54mm_Vertical, symbol Connector:Screw_Terminal_01x02
Connections:
- net GND: now also J10.1 (Pin_1), J7.1 (Pin_1), J8.1 (Pin_1), J9.1 (Pin_1)

Commit message: refresh
Connections:
- net +3.3V: now also J10.2 (Pin_2), J7.2 (Pin_2), J8.2 (Pin_2), J9.2 (Pin_2)
Changed lines of the file:
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@@
 	)
 	(junction
+		(at 135.89 156.21)
+		(diameter 0)
+		(color 0 0 0 0)
+	)
+	(junction
 		(at 181.61 73.66)
 		(diameter 0)
@@
 	)
 	(junction
+		(at 135.89 176.53)
+		(diameter 0)
+		(color 0 0 0 0)
+	)
+	(junction
 		(at 173.99 73.66)
 		(diameter 0)
@@
 	)
 	(junction
+		(at 135.89 166.37)
+		(diameter 0)
+		(color 0 0 0 0)
+	)
+	(junction
 		(at 173.99 66.04)
 		(diameter 0)
@@
 	(wire
 		(pts
+			(xy 135.89 176.53) (xy 135.89 186.69)
+		)
+		(stroke
+			(width 0)
+			(type default)
+		)
+	)
+	(wire
+		(pts
+			(xy 133.35 176.53) (xy 135.89 176.53)
+		)
+		(stroke
+			(width 0)
+			(type default)
+		)
+	)
+	(wire
+		(pts
 			(xy 262.89 111.76) (xy 276.86 111.76)
 		)
@@
 	(wire
 		(pts
+			(xy 135.89 166.37) (xy 135.89 176.53)
+		)
+		(stroke
+			(width 0)
+			(type default)
+		)
+	)
+	(wire
+		(pts
 			(xy 215.9 147.32) (xy 257.81 147.32)
 		)
@@
 	(wire
 		(pts
+			(xy 135.89 156.21) (xy 133.35 156.21)
+		)
+		(stroke
+			(width 0)
+			(type default)
+		)
+	)
+	(wire
+		(pts
 			(xy 227.33 190.5) (xy 153.67 190.5)
 		)
@@
 	(wire
 		(pts
+			(xy 133.35 186.69) (xy 135.89 186.69)
+		)
+		(stroke
+			(width 0)
+			(type default)
+		)
+	)
+	(wire
+		(pts
 			(xy 143.51 118.11) (xy 147.32 118.11)
 		)
@@
 	(wire
 		(pts
+			(xy 133.35 166.37) (xy 135.89 166.37)
+		)
+		(stroke
+			(width 0)
+			(type default)
+		)
+	)
+	(wire
+		(pts
 			(xy 119.38 156.21) (xy 116.84 156.21)
 		)
@@
 	(wire
 		(pts
+			(xy 135.89 156.21) (xy 135.89 166.37)
+		)
+		(stroke
+			(width 0)
+			(type default)
+		)
+	)
+	(wire
+		(pts
 			(xy 257.81 111.76) (xy 262.89 111.76)
 		)
@@
 					(unit 1)
 				)
+			)
+		)
+	)
+	(symbol
+		(lib_id "power:+3.3V")
+		(at 135.89 156.21 0)
+		(unit 1)
+		(body_style 1)
+		(exclude_from_sim no)
+		(in_bom yes)
+		(on_board yes)
+		(in_pos_files yes)
+		(dnp no)
+		(fields_autoplaced yes)
+		(property "Reference" "#PWR015"
+			(at 135.89 160.02 0)
+			(hide yes)
+			(show_name no)
+			(do_not_autoplace no)
+			(effects
+				(font
+					(size 1.27 1.27)
+				)
+			)
+		)
+		(property "Value" "+3.3V"
+			(at 135.89 151.13 0)
+			(show_name no)
+			(do_not_autoplace no)
+			(effects
+				(font
+					(size 1.27 1.27)
+				)
+			)
+		)
+		(property "Footprint" ""
+			(at 135.89 156.21 0)
+			(hide yes)
+			(show_name no)
+			(do_not_autoplace no)
+			(effects
+				(font
+					(size 1.27 1.27)
+				)
+			)
+		)
+		(property "Datasheet" ""
+			(at 135.89 156.21 0)
+			(hide yes)
+			(show_name no)
+			(do_not_autoplace no)
+			(effects
+				(font
+					(size 1.27 1.27)
+				)
+			)
+		)
+		(property "Description" "Power symbol creates a global label with name \"+3.3V\""
+			(at 135.89 156.21 0)
+			(hide yes)
+			(show_name no)
+			(do_not_autoplace no)
+			(effects
+				(font
+					(size 1.27 1.27)
+				)
+			)
+		)
+		(pin "1"
+		)
+		(instances
+			(project "micro"
+				(path "/20867279-5aff-4560-94cd-e855d560edf3"
+					(reference "#PWR015")
+					(unit 1)
+				)
