File: power/power.kicad_sch (KiCad schematic)
At the start: 11 parts, among them J1 XT30, J2 Screw_Terminal_01x02, J3 Screw_Terminal_01x02, J4 Screw_Terminal_01x02, J5 Screw_Terminal_01x02, J6 Screw_Terminal_01x02, J7 Screw_Terminal_01x02, J8 Screw_Terminal_01x02, J9 Screw_Terminal_01x02, U1 UC3843_SOIC8

Commit message: refresh
Parts:
- removed D1: 1N5820, Diode_THT:D_DO-201AD_P15.24mm_Horizontal, symbol Diode:1N5820
- removed J1: XT30, Connector_AMASS:AMASS_XT30U-F_1x02_P5.0mm_Vertical, symbol Connector:Screw_Terminal_01x02
- removed J2, J3, J4, J5, J6, J7, J8, J9: Screw_Terminal_01x02, Connector_PinHeader_2.54mm:PinHeader_1x02_P2.54mm_Vertical, symbol Connector:Screw_Terminal_01x02
- removed U1: UC3843_SOIC8, Package_SO:SOIC-8_3.9x4.9mm_P1.27mm, symbol Regulator_Controller:UC3843_SOIC8
- added C1, C2: C_Polarized, Capacitor_SMD:C_0805_2012Metric_Pad1.18x1.45mm_HandSolder, symbol Device:C_Polarized
- added J10, J11: Screw_Terminal_01x02, Connector_JST:JST_EH_B2B-EH-A_1x02_P2.50mm_Vertical, symbol Connector:Screw_Terminal_01x02
- added Q1, Q2: IRFZ44N, Package_TO_SOT_THT:TO-220-3_Vertical, symbol Transistor_FET:BUZ11
- added R1, R2, R3: R_US, Resistor_SMD:R_0805_2012Metric_Pad1.20x1.40mm_HandSolder, symbol Device:R_US
- added U2: (no value), Package_TO_SOT_SMD:SOT-23-6, symbol me:HY2120
Connections:
- net GND: now also Q2.3 (S), R2.2
- new net: Q2.1 (G), U2.2 (OC)
- new net: Q1.2 (D), Q2.2 (D)
- new net: R1.1, U2.5 (VDD)
- new net: C1.1, R1.2
- new net: C1.2, C2.2, J10.1 (Pin_1), Q1.3 (S), U2.6 (VSS)
- new net: J10.2 (Pin_2), J11.1 (Pin_1)
- new net: Q1.1 (G), U2.1 (OD)
- new net: R2.1, U2.3 (CS)
- new net: R3.1, U2.4 (VC)
- new net: C2.1, J11.2 (Pin_2), R3.2

Commit message: refresh
Parts:
- added C3: 10u, Capacitor_SMD:C_0805_2012Metric_Pad1.18x1.45mm_HandSolder, symbol Device:C_Polarized
- added C4: C, symbol Device:C
- added J1: Barrel_Jack_Switch, Connector_BarrelJack:BarrelJack_GCT_DCJ200-10-A_Horizontal, symbol Connector:Barrel_Jack_Switch
- added R4: 125, Resistor_SMD:R_0805_2012Metric_Pad1.20x1.40mm_HandSolder, symbol Device:R_US
- added R5: 715, Resistor_SMD:R_0805_2012Metric_Pad1.20x1.40mm_HandSolder, symbol Device:R_US
- added U1: LM317_SOT-223, Package_TO_SOT_SMD:SOT-223-3_TabPin2, symbol Regulator_Linear:LM317_SOT-223
Connections:
- net GND: now also C3.2, C4.2, J1.2, J1.3, R5.1
- net at C1.1, R1.2: now also J11.2 (Pin_2), C3.1, R4.2, U1.2 (VO)
- net at J10.2 (Pin_2), J11.1 (Pin_1): now also C2.1, R3.2
- new net: C4.1, J1.1, U1.3 (VI)
- new net: R4.1, R5.2, U1.1 (ADJ)

Commit message: refresh
Parts:
- removed C4: C, symbol Device:C
- removed J1: Barrel_Jack_Switch, Connector_BarrelJack:BarrelJack_GCT_DCJ200-10-A_Horizontal, symbol Connector:Barrel_Jack_Switch
- removed R4: 125, Resistor_SMD:R_0805_2012Metric_Pad1.20x1.40mm_HandSolder, symbol Device:R_US
- removed R5: 715, Resistor_SMD:R_0805_2012Metric_Pad1.20x1.40mm_HandSolder, symbol Device:R_US
- removed U1: LM317_SOT-223, Package_TO_SOT_SMD:SOT-223-3_TabPin2, symbol Regulator_Linear:LM317_SOT-223
