File: power/power.kicad_pcb (KiCad board)
At the start: 2 copper layers, 60 x 60 mm, 22 parts, among them J1 XT30, J2 JST Terminal, U1 AP63200WU, U2 AP63200WU

Commit message: refresh
Routing:
- net Net-(J2-Pin_3): track 88.8 -> 73.0 mm
- net Net-(J2-Pin_1): track 87.9 -> 72.0 mm

Commit message: refresh
Parts:
- removed C10: 100p, Capacitor_THT:C_Disc_D4.3mm_W1.9mm_P5.00mm
- removed C11, C12: 22u, Capacitor_THT:CP_Radial_D5.0mm_P2.50mm
- removed C7, C8: 10u, Capacitor_THT:CP_Radial_D5.0mm_P2.50mm
- removed C9: 100n, Capacitor_THT:C_Disc_D4.3mm_W1.9mm_P5.00mm
- removed L2: L, Inductor_SMD:L_Wuerth_HCI-1890
- removed R3: 52.3k, Resistor_THT:R_Axial_DIN0204_L3.6mm_D1.6mm_P2.54mm_Vertical
- removed R4: 10k, Resistor_THT:R_Axial_DIN0204_L3.6mm_D1.6mm_P2.54mm_Vertical
- removed U2: AP63200WU, Package_TO_SOT_SMD:TSOT-23-6
- added J3: Screw_Terminal_01x02, Connector_PinHeader_2.54mm:PinHeader_1x02_P2.54mm_Vertical, F.Cu at (97.8, 84.6)
- added J4: Screw_Terminal_01x02, Connector_PinHeader_2.54mm:PinHeader_1x02_P2.54mm_Vertical, F.Cu at (102.3, 84.6)
- added J5: Screw_Terminal_01x02, Connector_PinHeader_2.54mm:PinHeader_1x02_P2.54mm_Vertical, F.Cu at (106.9, 84.6)
- added J6: Screw_Terminal_01x02, Connector_PinHeader_2.54mm:PinHeader_1x02_P2.54mm_Vertical, F.Cu at (111.5, 84.6)
- added J7: Screw_Terminal_01x02, Connector_PinHeader_2.54mm:PinHeader_1x02_P2.54mm_Vertical, F.Cu at (116.1, 84.6)
- added J8: Screw_Terminal_01x02, Connector_PinHeader_2.54mm:PinHeader_1x02_P2.54mm_Vertical, F.Cu at (120.7, 84.6)
- added J9: Screw_Terminal_01x02, Connector_PinHeader_2.54mm:PinHeader_1x02_P2.54mm_Vertical, F.Cu at (125.3, 84.6)
- J2: value JST Terminal -> Screw_Terminal_01x02; footprint Connector_JST:JST_PH_B3B-PH-K_1x03_P2.00mm_Vertical -> Connector_PinHeader_2.54mm:PinHeader_1x02_P2.54mm_Vertical
- L1: value L -> 6.8u
- moved C6 125.7 mm to (84.9, 133.9), turned to 0 degrees
- moved J2 111.5 mm to (93.2, 84.6), turned to 0 degrees
- moved C5 106.4 mm to (89.6, 140.3), turned to 0 degrees
- moved R1 87.2 mm to (77.8, 78.5), turned to 0 degrees
- moved R2 84.1 mm to (77.8, 81.6), turned to 0 degrees
- moved C2 83.2 mm to (84.9, 120.8), turned to 0 degrees
- moved C1 75.2 mm to (84.9, 114.2), turned to 0 degrees
- moved C3 74.1 mm to (96.7, 72.2), turned to 0 degrees
- moved C4 71.9 mm to (96.7, 75.6), turned to 0 degrees
- moved L1 68.0 mm to (138.8, 128.0)
- moved U1 67.9 mm to (126.3, 128.8), turned to -90 degrees
- moved J1 58.7 mm to (114.3, 128.0)
Connections:
- R1 pad 1: Net-(J2-Pin_1) -> Net-(U1-FB)
- R1 pad 2: Net-(U1-FB) -> Net-(J2-Pin_1)
- R2 pad 1: Net-(U1-FB) -> GND
- R2 pad 2: GND -> Net-(U1-FB)
Routing:
- net Net-(J1-Pin_2): track 326.1 -> 0.00 mm
- net Net-(J2-Pin_3): track 73.0 -> 0.00 mm
- net Net-(J2-Pin_1): track 72.0 -> 0.00 mm
- net Net-(U2-FB): track 18.8 -> 0.00 mm
- net Net-(U1-FB): track 18.6 -> 0.00 mm
- net Net-(U2-SW): track 16.7 -> 0.00 mm
- net Net-(U1-SW): track 16.4 -> 0.00 mm
- net Net-(U2-BST): track 2.43 -> 0.00 mm
- net Net-(U1-BST): track 2.19 -> 0.00 mm
- added copper zone on F.Cu, net Net-(J1-Pin_2)
- removed copper zone on B.Cu, net GND
- removed copper zone on F.Cu, net GND

Commit message: refresh
Parts:
- removed C3: 100n, Capacitor_THT:C_Disc_D4.3mm_W1.9mm_P5.00mm
- removed C4: 100p, Capacitor_THT:C_Disc_D4.3mm_W1.9mm_P5.00mm
- removed C5, C6: 22u, Capacitor_THT:CP_Radial_D5.0mm_P2.50mm
- removed J1: XT30, Connector_AMASS:AMASS_XT30U-F_1x02_P5.0mm_Vertical
- removed J2, J3, J4, J5, J6, J7, J8, J9: Screw_Terminal_01x02, Connector_PinHeader_2.54mm:PinHeader_1x02_P2.54mm_Vertical
- removed L1: 6.8u, Inductor_SMD:L_Wuerth_HCI-1890
- removed U1: AP63200WU, Package_TO_SOT_SMD:TSOT-23-6
- added J10: Screw_Terminal_01x02, Connector_JST:JST_EH_B2B-EH-A_1x02_P2.50mm_Vertical, F.Cu at (95.4, 93.9)
- added J11: Screw_Terminal_01x02, Connector_JST:JST_EH_B2B-EH-A_1x02_P2.50mm_Vertical, F.Cu at (95.4, 103.3)
- added Q1: IRFZ44N, Package_TO_SOT_THT:TO-220-3_Vertical, F.Cu at (106.5, 93.8)
- added Q2: IRFZ44N, Package_TO_SOT_THT:TO-220-3_Vertical, F.Cu at (111.6, 105.9)
- added R3: R_US, Resistor_SMD:R_0805_2012Metric_Pad1.20x1.40mm_HandSolder, B.Cu at (99.4, 103.1)
- added U2: ~, Package_TO_SOT_SMD:SOT-23-6, B.Cu at (101.5, 99.8)
- C1, C2: value 10u -> C_Polarized; footprint Capacitor_THT:CP_Radial_D5.0mm_P2.50mm -> Capacitor_SMD:C_0805_2012Metric_Pad1.18x1.45mm_HandSolder; moved to B.Cu
- R1: value 31.6k -> R_US; footprint Resistor_THT:R_Axial_DIN0204_L3.6mm_D1.6mm_P2.54mm_Vertical -> Resistor_SMD:R_0805_2012Metric_Pad1.20x1.40mm_HandSolder
- R2: value 10.2k -> R_US; footprint Resistor_THT:R_Axial_DIN0204_L3.6mm_D1.6mm_P2.54mm_Vertical -> Resistor_SMD:R_0805_2012Metric_Pad1.20x1.40mm_HandSolder; moved to B.Cu
- moved R2 35.1 mm to (106.5, 101.8), turned to -90 degrees
- moved R1 30.6 mm to (99.7, 99.8)
- moved C1 26.8 mm to (101.1, 92.9), turned to -90 degrees
- moved C2 21.4 mm to (101.1, 106.9), turned to -90 degrees
Connections:
- C1 pad 1: Net-(J1-Pin_2) -> Net-(C1-Pad1)
- C1 pad 2: GND -> Net-(J10-Pin_1)
- C2 pad 1: Net-(J1-Pin_2) -> Net-(J11-Pin_2)
- C2 pad 2: GND -> Net-(J10-Pin_1)
- R1 pad 1: Net-(U1-FB) -> Net-(U2-VDD)
- R1 pad 2: Net-(J2-Pin_1) -> Net-(C1-Pad1)
- R2 pad 1: GND -> Net-(U2-CS)
- R2 pad 2: Net-(U1-FB) -> GND
Routing:
- net Net-(J10-Pin_1): track 0.00 -> 25.2 mm
- net Net-(Q2-G): track 0.00 -> 13.6 mm, vias 0 -> 1
- net Net-(Q1-D): track 0.00 -> 12.1 mm
- net Net-(C1-Pad1): track 0.00 -> 8.10 mm, vias 0 -> 1
- net Net-(Q1-G): track 0.00 -> 7.51 mm
- net Net-(U2-CS): track 0.00 -> 3.86 mm
- net Net-(U2-VC): track 0.00 -> 2.02 mm
- net Net-(U2-VDD): track 0.00 -> 1.65 mm, vias 0 -> 1
- added copper zone on B.Cu, net GND
- added copper zone on F.Cu, net GND
- added copper zone on B.Cu, net Net-(J10-Pin_1)
- added copper zone on B.Cu, net Net-(J10-Pin_2)
- added copper zone on B.Cu, net Net-(J11-Pin_2)
- removed copper zone on F.Cu, net Net-(J1-Pin_2)

Commit message: refresh
Parts:
- added C3: 10u, Capacitor_SMD:C_0805_2012Metric_Pad1.18x1.45mm_HandSolder, F.Cu at (65.8, 113.2)
- added J1: Barrel_Jack_Switch, Connector_BarrelJack:BarrelJack_GCT_DCJ200-10-A_Horizontal, F.Cu at (120.7, 78.5)
- added R4: 125, Resistor_SMD:R_0805_2012Metric_Pad1.20x1.40mm_HandSolder, F.Cu at (61.0, 113.1)
- added R5: 715, Resistor_SMD:R_0805_2012Metric_Pad1.20x1.40mm_HandSolder, F.Cu at (61.0, 116.1)
- added U1: LM317_SOT-223, Package_TO_SOT_SMD:SOT-223-3_TabPin2, F.Cu at (115.8, 117.7)
- C1, C2, R2, R3, U2: moved to F.Cu
- moved U2 13.8 mm to (103.4, 113.5), turned to 0 degrees
- turned R3 to 0 degrees
Connections:
- C1 pad 1: Net-(C1-Pad1) -> Net-(J11-Pin_2)
- C2 pad 1: Net-(J11-Pin_2) -> Net-(J10-Pin_2)
- R1 pad 2: Net-(C1-Pad1) -> Net-(J11-Pin_2)
- R3 pad 2: Net-(J11-Pin_2) -> Net-(J10-Pin_2)
Routing:
- net Net-(J10-Pin_1): track 25.2 -> 0.00 mm
- net GND: track 0.00 -> 20.6 mm
- net Net-(Q2-G): track 13.6 -> 0.00 mm
- net Net-(Q1-D): track 12.1 -> 0.00 mm
- net Net-(C1-Pad1): track 8.10 -> 0.00 mm, vias 1 -> 0
- net Net-(Q1-G): track 7.51 -> 0.00 mm
- net Net-(U2-CS): track 3.86 -> 0.00 mm
- net Net-(U2-VC): track 2.02 -> 0.00 mm
- net Net-(U2-VDD): track 1.65 -> 0.00 mm
- removed copper zone on B.Cu, net Net-(J10-Pin_1)
- removed copper zone on B.Cu, net Net-(J10-Pin_2)
- removed copper zone on B.Cu, net Net-(J11-Pin_2)
