File: power/power.kicad_pcb (KiCad board)
At the start: 2 copper layers, 60 x 60 mm, 15 parts, among them J1 Barrel_Jack_Switch, J10 Screw_Terminal_01x02, J11 Screw_Terminal_01x02, Q1 IRFZ44N, Q2 IRFZ44N, U1 LM317_SOT-223

Commit message: refresh
Parts:
- removed C1, C2: C_Polarized, Capacitor_SMD:C_0805_2012Metric_Pad1.18x1.45mm_HandSolder
- removed C3: 10u, Capacitor_SMD:C_0805_2012Metric_Pad1.18x1.45mm_HandSolder
- removed J1: Barrel_Jack_Switch, Connector_BarrelJack:BarrelJack_GCT_DCJ200-10-A_Horizontal
- removed J10, J11: Screw_Terminal_01x02, Connector_JST:JST_EH_B2B-EH-A_1x02_P2.50mm_Vertical
- removed Q1, Q2: IRFZ44N, Package_TO_SOT_THT:TO-220-3_Vertical
- removed R1, R2, R3: R_US, Resistor_SMD:R_0805_2012Metric_Pad1.20x1.40mm_HandSolder
- removed U1: LM317_SOT-223, Package_TO_SOT_SMD:SOT-223-3_TabPin2
- added C10: 100nf/50V, Capacitor_SMD:C_0402_1005Metric_Pad0.74x0.62mm_HandSolder, F.Cu at (87.4, 123.5)
- added C11: 100nf/50V, Capacitor_SMD:C_0402_1005Metric_Pad0.74x0.62mm_HandSolder, F.Cu at (87.4, 125.5)
- added C15: 22uf/10V, A_HDJ_Library:C_0603_1608Metric, F.Cu at (75.8, 122.1)
- added C16: 22uf/10V, A_HDJ_Library:C_0603_1608Metric, F.Cu at (79.8, 112.1)
- added C17: 22uf/10V, A_HDJ_Library:C_0603_1608Metric, F.Cu at (79.8, 114.6)
- added C18: 22uf/10V, A_HDJ_Library:C_0603_1608Metric, F.Cu at (79.8, 117.1)
- added C19: 100uf/10V, A_HDJ_Library:C_0603_1608Metric, F.Cu at (79.8, 119.6)
- added C20: 22uf/10V, A_HDJ_Library:C_0603_1608Metric, F.Cu at (79.8, 122.1)
- added C21: 22uf/10V, A_HDJ_Library:C_0603_1608Metric, F.Cu at (83.8, 112.1)
- added C22: 22uf/10V, A_HDJ_Library:C_0603_1608Metric, F.Cu at (83.8, 114.6)
- added C23: 22uf/10V, A_HDJ_Library:C_0603_1608Metric, F.Cu at (83.8, 117.1)
- added C24: 100uf/10V, A_HDJ_Library:C_0603_1608Metric, F.Cu at (83.8, 119.6)
- added C4: C_Polarized, Capacitor_SMD:C_0805_2012Metric_Pad1.18x1.45mm_HandSolder, F.Cu at (94.4, 103.1)
- added C5: C_Polarized, Capacitor_SMD:C_0805_2012Metric_Pad1.18x1.45mm_HandSolder, F.Cu at (94.4, 106.1)
- added C6: 22uf/10V, A_HDJ_Library:C_0603_1608Metric, F.Cu at (75.8, 112.1)
- added C7: 22uf/10V, A_HDJ_Library:C_0603_1608Metric, F.Cu at (75.8, 114.6)
- added C8: 22uf/10V, A_HDJ_Library:C_0603_1608Metric, F.Cu at (75.8, 117.1)
- added C9: 22uf/10V, A_HDJ_Library:C_0603_1608Metric, F.Cu at (75.8, 119.6)
- added J12: Screw_Terminal_01x02, Connector_JST:JST_EH_B2B-EH-A_1x02_P2.50mm_Vertical, F.Cu at (89.3, 113.4)
- added J13: Screw_Terminal_01x02, Connector_JST:JST_EH_B2B-EH-A_1x02_P2.50mm_Vertical, F.Cu at (89.3, 119.3)
- added L1: 2.2uH/4.3A, Inductor_THT:L_Toroid_Vertical_L10.0mm_W5.0mm_P5.08mm, F.Cu at (120.0, 115.3)
- added L2: 2.2uH/4.3A, Inductor_THT:L_Toroid_Vertical_L10.0mm_W5.0mm_P5.08mm, F.Cu at (133.0, 115.4)
- added Q4: Q_NMOS, Package_TO_SOT_THT:TO-247-3_Horizontal_TabDown, F.Cu at (109.8, 107.8)
- added Q5: Q_NMOS, Package_TO_SOT_THT:TO-247-3_Horizontal_TabDown, F.Cu at (137.2, 107.8)
- added R10: R_US, Resistor_SMD:R_0805_2012Metric_Pad1.20x1.40mm_HandSolder, F.Cu at (94.4, 100.2)
- added R6: R_US, Resistor_SMD:R_0805_2012Metric_Pad1.20x1.40mm_HandSolder, F.Cu at (94.4, 88.4)
- added R7: R_US, Resistor_SMD:R_0805_2012Metric_Pad1.20x1.40mm_HandSolder, F.Cu at (94.4, 91.3)
- added R8: R_US, Resistor_SMD:R_0805_2012Metric_Pad1.20x1.40mm_HandSolder, F.Cu at (94.4, 94.3)
- added R9: R_US, Resistor_SMD:R_0805_2012Metric_Pad1.20x1.40mm_HandSolder, F.Cu at (94.4, 97.2)
- added U3: LM2734X, Package_TO_SOT_SMD:TSOT-23-6, F.Cu at (71.2, 117.8)
- added U4: LM2734X, Package_TO_SOT_SMD:TSOT-23-6, F.Cu at (71.2, 122.5)
- R4: value 125 -> R_US
- R5: value 715 -> R_US
- moved R4 45.3 mm to (94.4, 82.5)
- moved R5 45.3 mm to (94.4, 85.4)
- moved U2 32.2 mm to (71.2, 113.2)
Connections:
- R4 pad 1: Net-(U1-ADJ) -> Net-(U2-VDD)
- R4 pad 2: Net-(J11-Pin_2) -> PB+
- R5 pad 1: GND -> Net-(U2-VC)
- R5 pad 2: Net-(U1-ADJ) -> Net-(J12-Pin_2)
Routing:
- net GND: track 20.6 -> 0.00 mm
- net Net-(U2-VDD): vias 1 -> 0
- net Net-(U2-OC): vias 1 -> 0
- removed copper zone on B.Cu, net GND
- removed copper zone on F.Cu, net GND
